Commit message: fix: align v0.4 geometry and add gamepad teleop

File: robot_description/xlerobot_v04.urdf (robot description, URDF)
Before this commit: robot xlerobot_v04_servo_dualwheel, 22 links, 21 joints
Links:
- link head_tilt_link: geometry visual box size=0.020 0.070 0.054; visual cylinder length=0.010 radius=0.008
Joints:
- joint head_camera_joint: origin xyz=0.025 0 0.03 rpy=-1.5708 0 -1.5708 -> xyz=0.083 0 0.005 rpy=-1.5708 0 -1.5708
- joint left_wheel_joint: origin xyz=-0.15 0.125 -0.3065 rpy=0 0 0 -> xyz=-0.15 0.23 -0.3065 rpy=0 0 0
- joint right_wheel_joint: origin xyz=-0.15 -0.125 -0.3065 rpy=0 0 0 -> xyz=-0.15 -0.23 -0.3065 rpy=0 0 0

Commit message: fix: expose v0.4 tires and relocate drive covers

File: robot_description/xlerobot_v04.urdf (robot description, URDF)
Before this commit: robot xlerobot_v04_servo_dualwheel, 22 links, 21 joints
Links:
- link base_link: geometry collision box size=0.315 0.405 0.59; collision box size=0.3913 0.459 0.10
- link left_wheel_link: geometry collision cylinder length=0.05 radius=0.0635; visual cylinder length=0.05 radius=0.0635
- link right_wheel_link: geometry collision cylinder length=0.05 radius=0.0635; visual cylinder length=0.05 radius=0.0635
Joints:
- joint left_wheel_joint: origin xyz=-0.15 0.23 -0.3065 rpy=0 0 0 -> xyz=-0.15 0.25 -0.3065 rpy=0 0 0
- joint right_wheel_joint: origin xyz=-0.15 -0.23 -0.3065 rpy=0 0 0 -> xyz=-0.15 -0.25 -0.3065 rpy=0 0 0

Commit message: fix: face neck camera toward v0.4 operating side

File: robot_description/xlerobot_v04.urdf (robot description, URDF)
Before this commit: robot xlerobot_v04_servo_dualwheel, 22 links, 21 joints
Joints:
- joint head_camera_joint: origin xyz=0.083 0 0.005 rpy=-1.5708 0 -1.5708 -> xyz=-0.083 0 0.005 rpy=-1.5708 0 1.5708

Commit message: fix: align v0.4 workspace and neck camera

File: robot_description/xlerobot_v04.urdf (robot description, URDF)
Before this commit: robot xlerobot_v04_servo_dualwheel, 22 links, 21 joints
Links:
- link head_tilt_link: geometry visual box size=0.004 0.068 0.050; visual box size=0.020 0.074 0.056

Commit message: physics: ground v0.4 parameters in official datasheets

File: robot_description/xlerobot_v04.urdf (robot description, URDF)
Before this commit: robot xlerobot_v04_servo_dualwheel, 22 links, 21 joints
Joints:
- joint Elbow_L: limit lower=-0.22 upper=3.14 effort=3.35 velocity=4.0 -> lower=-0.22 upper=3.14 effort=2.94 velocity=4.0
- joint Elbow_R: limit lower=-0.22 upper=3.14 effort=3.35 velocity=4.0 -> lower=-0.22 upper=3.14 effort=2.94 velocity=4.0
- joint Jaw_L: limit lower=-0.37453 upper=1.74533 effort=10 velocity=4.0 -> lower=-0.37453 upper=1.74533 effort=2.94 velocity=4.0
- joint Jaw_R: limit lower=-0.37453 upper=1.74533 effort=10 velocity=4.0 -> lower=-0.37453 upper=1.74533 effort=2.94 velocity=4.0
- joint Pitch_L: limit lower=-0.22 upper=3.37 effort=3.35 velocity=4.0 -> lower=-0.22 upper=3.37 effort=2.94 velocity=4.0
- joint Pitch_R: limit lower=-0.22 upper=3.37 effort=3.35 velocity=4.0 -> lower=-0.22 upper=3.37 effort=2.94 velocity=4.0
- joint Rotation_L: limit lower=-2.16 upper=2.16 effort=3.35 velocity=4.0 -> lower=-2.16 upper=2.16 effort=2.94 velocity=4.0
- joint Rotation_R: limit lower=-2.16 upper=2.16 effort=3.35 velocity=4.0 -> lower=-2.16 upper=2.16 effort=2.94 velocity=4.0
- joint Wrist_Pitch_L: limit lower=-1.65806 upper=1.65806 effort=3.35 velocity=4.0 -> lower=-1.65806 upper=1.65806 effort=2.94 velocity=4.0
- joint Wrist_Pitch_R: limit lower=-1.65806 upper=1.65806 effort=3.35 velocity=4.0 -> lower=-1.65806 upper=1.65806 effort=2.94 velocity=4.0
- joint Wrist_Roll_L: limit lower=-2.74385 upper=2.84121 effort=3.35 velocity=4.0 -> lower=-2.74385 upper=2.84121 effort=2.94 velocity=4.0
- joint Wrist_Roll_R: limit lower=-2.74385 upper=2.84121 effort=3.35 velocity=4.0 -> lower=-2.74385 upper=2.84121 effort=2.94 velocity=4.0
